File: servicetastatur.kicad_pcb (KiCad board)
At the start: 2 copper layers, 106 x 57 mm, 11 parts, among them J1 Conn_01x16_Socket, J2 Conn_01x06_Socket, U1 AT24CS16-SSHM, U2 TL7705A, U3 74HC165, U4 74HC00, U5 MC34063AP, U6 27C128, Y1 Crystal

Commit message: gross
Parts:
- moved Y1 6.04 mm to (94.5, 82.0)
- moved U6 5.49 mm to (77.0, 120.5)
- moved C2 4.74 mm to (115.5, 113.5)
- moved U4 4.08 mm to (80.3, 97.0)
- moved C1 4.03 mm to (116.0, 106.5)
- moved U1 2.79 mm to (124.9, 82.5)
- moved U2 2.56 mm to (156.0, 82.5)
- moved U5 2.35 mm to (135.4, 131.5)
- moved J2 0.50 mm to (151.0, 84.5)
Other:
- board size 106 x 57 mm -> 113 x 60 mm

Commit message: sdfsdf
Parts:
- added C3: C, Capacitor_THT:C_Axial_L3.8mm_D2.6mm_P7.50mm_Horizontal, F.Cu at (122.0, 105.0)
- added C4: C, Capacitor_THT:C_Axial_L3.8mm_D2.6mm_P7.50mm_Horizontal, F.Cu at (84.0, 87.0)
- added C5: C, Capacitor_THT:C_Axial_L3.8mm_D2.6mm_P7.50mm_Horizontal, F.Cu at (136.0, 82.5)
- added C6: C, Capacitor_THT:C_Axial_L3.8mm_D2.6mm_P7.50mm_Horizontal, F.Cu at (142.0, 80.2)
- added C7: C, Capacitor_THT:C_Axial_L3.8mm_D2.6mm_P7.50mm_Horizontal, F.Cu at (146.0, 131.5)
- added R1: 3.3 kΩ ±5%, Resistor_THT:R_Axial_DIN0207_L6.3mm_D2.5mm_P10.16mm_Horizontal, F.Cu at (89.3, 131.0)
- added R2: 22 Ω ±5%, Resistor_THT:R_Axial_DIN0207_L6.3mm_D2.5mm_P10.16mm_Horizontal, F.Cu at (102.3, 131.0)
- added R3: 110 Ω ±1%, Resistor_THT:R_Axial_DIN0207_L6.3mm_D2.5mm_P10.16mm_Horizontal, F.Cu at (118.3, 118.7)
- added R4: 3.3 kΩ ±5%, Resistor_THT:R_Axial_DIN0207_L6.3mm_D2.5mm_P10.16mm_Horizontal, F.Cu at (118.3, 121.5)
- added R5: 270 Ω ±5%, Resistor_THT:R_Axial_DIN0207_L6.3mm_D2.5mm_P10.16mm_Horizontal, F.Cu at (118.3, 124.0)
- J1: value Conn_01x16_Socket -> Conn_02x08_Odd_Even; footprint Connector_Molex:Molex_Picoflex_90325-0016_2x08_P1.27mm_Vertical -> Connector_PinSocket_1.00mm:PinSocket_1x16_P1.00mm_Vertical_SMD_Pin1Right; moved to B.Cu
- moved J1 2.74 mm to (102.0, 127.0)
- moved C2 1.12 mm to (116.5, 113.0)
- moved Y1 1.12 mm to (95.0, 83.0)
- moved C1 0.71 mm to (116.5, 106.0)
- moved U6 0.71 mm to (77.5, 120.0)
Connections:
- U1 pad 4: unconnected-(U1-GND-Pad4) -> GND
- U1 pad 8: unconnected-(U1-VCC-Pad8) -> Net-(U1-VCC)
- U2 pad 4: unconnected-(U2-GND-Pad4) -> GND
- U2 pad 8: unconnected-(U2-VCC-Pad8) -> Net-(U2-VCC)
- U3 pad 16: unconnected-(U3-VCC-Pad16) -> Net-(U3-VCC)
- U3 pad 8: unconnected-(U3-GND-Pad8) -> GND
- U4 pad 14: unconnected-(U4E-VCC-Pad14) -> Net-(U4E-VCC)
- U4 pad 7: unconnected-(U4E-GND-Pad7) -> GND
- U5 pad 4: unconnected-(U5-GND-Pad4) -> GND
- U5 pad 6: unconnected-(U5-Vin-Pad6) -> Net-(U5-Vin)
- U6 pad 14: unconnected-(U6-GND-Pad14) -> GND
Other:
- outline, holes or cut-outs redrawn

Commit message: CPU
Parts:
- added C8: C, Capacitor_THT:CP_Radial_Tantal_D4.5mm_P2.50mm, F.Cu at (88.8, 74.4)
- added C9: C, Capacitor_THT:CP_Radial_Tantal_D4.5mm_P2.50mm, F.Cu at (88.8, 85.5)
- added D1: D, Diode_THT:D_DO-15_P15.24mm_Horizontal, F.Cu at (114.8, 116.5)
- added D2: D, Diode_THT:D_DO-15_P15.24mm_Horizontal, F.Cu at (117.8, 127.8)
- added R6: R, Resistor_THT:R_Axial_DIN0414_L11.9mm_D4.5mm_P15.24mm_Horizontal, F.Cu at (117.5, 131.8)
- added U7: ~, Package_LCC:PLCC-44_THT-Socket, F.Cu at (115.5, 86.3)
- moved J1 0.93 mm to (102.8, 127.5)
- moved R3 0.90 mm to (117.6, 119.2)
- moved R4 0.90 mm to (117.6, 122.0)
- moved R5 0.90 mm to (117.6, 124.5)
- moved Y1 0.50 mm to (95.0, 82.5)
- moved C4 0.35 mm to (83.8, 86.8)
- moved R1 0.35 mm to (89.1, 131.2)
- moved R2 0.35 mm to (102.1, 131.2)
- moved U4 0.25 mm to (80.0, 97.0)
Connections:
- C1 pad 2: unconnected-(C1-Pad2) -> GND
- C2 pad 2: unconnected-(C2-Pad2) -> GND
- C3 pad 2: Net-(U3-VCC) -> VCC
- C4 pad 2: Net-(U4E-VCC) -> VCC
- C6 pad 1: GND -> Net-(U1-WP)
- C6 pad 2: Net-(U2-VCC) -> unconnected-(C6-Pad2)
- R3 pad 2: unconnected-(R3-Pad2) -> Net-(R3-Pad2)
- R4 pad 2: unconnected-(R4-Pad2) -> Net-(R3-Pad2)
- U1 pad 7: unconnected-(U1-WP-Pad7) -> Net-(U1-WP)
- U2 pad 8: Net-(U2-VCC) -> unconnected-(U2-VCC-Pad8)
- U3 pad 11: unconnected-(U3-D0-Pad11) -> D0
- U3 pad 12: unconnected-(U3-D1-Pad12) -> D1
- U3 pad 13: unconnected-(U3-D2-Pad13) -> D2
- U3 pad 14: unconnected-(U3-D3-Pad14) -> D3
- U3 pad 16: Net-(U3-VCC) -> VCC
- U3 pad 3: unconnected-(U3-D4-Pad3) -> D4
- U3 pad 4: unconnected-(U3-D5-Pad4) -> D5
- U3 pad 5: unconnected-(U3-D6-Pad5) -> D6
- U3 pad 6: unconnected-(U3-D7-Pad6) -> D7
- U4 pad 10: unconnected-(U4-Pad10) -> Net-(U7-P3.6/WR)
- U4 pad 11: unconnected-(U4-Pad11) -> Net-(U7-P3.2/INT0)
- U4 pad 12: unconnected-(U4-Pad12) -> GND
- U4 pad 14: Net-(U4E-VCC) -> VCC
- U4 pad 9: unconnected-(U4-Pad9) -> Net-(U7-P3.7/RD)
- U5 pad 1: unconnected-(U5-SwC-Pad1) -> Net-(U5-SwC)
- U6 pad 11: unconnected-(U6-D0-Pad11) -> D0
- U6 pad 12: unconnected-(U6-D1-Pad12) -> D1
- U6 pad 13: unconnected-(U6-D2-Pad13) -> D2
- U6 pad 15: unconnected-(U6-D3-Pad15) -> D3
- U6 pad 16: unconnected-(U6-D4-Pad16) -> D4
- U6 pad 17: unconnected-(U6-D5-Pad17) -> D5
- U6 pad 18: unconnected-(U6-D6-Pad18) -> D6
- U6 pad 19: unconnected-(U6-D7-Pad19) -> D7
- U6 pad 20: unconnected-(U6-~{CE}-Pad20) -> Net-(U6-~{CE})
- U6 pad 28: unconnected-(U6-VCC-Pad28) -> VCC
- Y1 pad 1: unconnected-(Y1-Pad1) -> Net-(U7-XTAL1)
- Y1 pad 2: unconnected-(Y1-Pad2) -> Net-(U7-XTAL2)
Routing:
- net D0: track 0.00 -> 68.3 mm
- net D1: track 0.00 -> 58.7 mm, vias 0 -> 2
- net D2: track 0.00 -> 51.7 mm, vias 0 -> 3
- net D7: track 0.00 -> 49.5 mm, vias 0 -> 3
- net Net-(U7-P3.2/INT0): track 0.00 -> 44.7 mm
- net D3: track 0.00 -> 40.9 mm, vias 0 -> 2
- net D6: track 0.00 -> 32.6 mm, vias 0 -> 2
- net VCC: track 0.00 -> 26.7 mm
- net Net-(U7-P3.6/WR): track 0.00 -> 26.1 mm
- net D4: track 0.00 -> 24.0 mm, vias 0 -> 1
- net Net-(U7-P3.7/RD): track 0.00 -> 23.7 mm
- net GND: track 0.00 -> 21.1 mm
- net (no net): track 0.00 -> 18.4 mm
- net Net-(U1-WP): track 0.00 -> 18.0 mm
- net unconnected-(D1-A-Pad2): track 0.00 -> 17.9 mm, vias 0 -> 1
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- added copper zone on B.Cu, net GND
Other:
- board text added: "8320/00020f/DN"
- board text added: "stwirtxt"

Commit message: anschluss
Parts:
- added C10: C, Capacitor_THT:CP_Radial_Tantal_D4.5mm_P2.50mm, F.Cu at (166.8, 77.8)
- added C11: C, Capacitor_THT:CP_Radial_Tantal_D4.5mm_P2.50mm, F.Cu at (151.8, 77.2)
- added D3: D, Diode_THT:D_DO-15_P15.24mm_Horizontal, F.Cu at (168.0, 114.0)
- added J3: Conn_01x06, ConnPad:Conn01x06, F.Cu at (182.2, 103.2)
- added R10: 1 kΩ ±1%, Resistor_THT:R_Axial_DIN0207_L6.3mm_D2.5mm_P10.16mm_Horizontal, F.Cu at (168.1, 102.2)
- added R11: 10 kΩ ±5%, Resistor_THT:R_Axial_DIN0207_L6.3mm_D2.5mm_P10.16mm_Horizontal, F.Cu at (166.6, 83.5)
- added R12: 22 Ω ±5%, Resistor_THT:R_Axial_DIN0207_L6.3mm_D2.5mm_P10.16mm_Horizontal, F.Cu at (148.8, 74.5)
- added R13: 47 kΩ ±5%, Resistor_THT:R_Axial_DIN0207_L6.3mm_D2.5mm_P10.16mm_Horizontal, F.Cu at (138.6, 77.2)
- added R14: 1 kΩ ±1%, Resistor_THT:R_Axial_DIN0207_L6.3mm_D2.5mm_P10.16mm_Horizontal, F.Cu at (122.5, 93.4)
- added R15: 4.7 kΩ ±1%, Resistor_THT:R_Axial_DIN0207_L6.3mm_D2.5mm_P10.16mm_Horizontal, F.Cu at (168.2, 97.1)
- added R16: 47 Ω ±1%, Resistor_THT:R_Axial_DIN0207_L6.3mm_D2.5mm_P10.16mm_Horizontal, F.Cu at (168.2, 99.5)
- added R17: 270 Ω ±5%, Resistor_THT:R_Axial_DIN0207_L6.3mm_D2.5mm_P10.16mm_Horizontal, F.Cu at (168.0, 105.0)
- added R18: 270 Ω ±5%, Resistor_THT:R_Axial_DIN0207_L6.3mm_D2.5mm_P10.16mm_Horizontal, F.Cu at (168.0, 107.5)
- added R7: 1 kΩ ±1%, Resistor_THT:R_Axial_DIN0207_L6.3mm_D2.5mm_P10.16mm_Horizontal, F.Cu at (166.6, 86.2)
- added R8: 1 kΩ ±1%, Resistor_THT:R_Axial_DIN0207_L6.3mm_D2.5mm_P10.16mm_Horizontal, F.Cu at (166.6, 88.8)
- added R9: 1 kΩ ±1%, Resistor_THT:R_Axial_DIN0207_L6.3mm_D2.5mm_P10.16mm_Horizontal, F.Cu at (166.6, 91.8)
Connections:
- C6 pad 1: Net-(U1-WP) -> GND
- C6 pad 2: unconnected-(C6-Pad2) -> Net-(U2-REF)
- U1 pad 7: Net-(U1-WP) -> GND
- U2 pad 1: unconnected-(U2-REF-Pad1) -> Net-(U2-REF)
- U2 pad 2: unconnected-(U2-~{RESIN}-Pad2) -> Net-(U2-~{RESIN})
- U2 pad 7: unconnected-(U2-SENSE-Pad7) -> Net-(U2-SENSE)
- U2 pad 8: unconnected-(U2-VCC-Pad8) -> Net-(U2-SENSE)
- U7 pad 1: unconnected-(U7-Vss1-Pad1) -> GND
- U7 pad 22: unconnected-(U7-Vss-Pad22) -> GND
Routing:
- net Net-(J3-Pin_5): track 0.00 -> 55.3 mm
- net GND: track 21.1 -> 74.4 mm
- net Net-(J3-Pin_4): track 0.00 -> 44.4 mm
- net Net-(J3-Pin_3): track 0.00 -> 30.1 mm
- net Net-(U1-VCC): track 0.00 -> 21.9 mm, vias 0 -> 1
- net Net-(U1-WP): track 18.0 -> 0.00 mm
- net Net-(R11-Pad2): track 0.00 -> 17.8 mm
- net Net-(C11-Pad2): track 0.00 -> 17.3 mm
- net Net-(U2-SENSE): track 0.00 -> 15.9 mm
- net Net-(U2-~{RESIN}): track 0.00 -> 9.93 mm
- net unconnected-(J2-Pin_6-Pad6): track 0.00 -> 9.87 mm, vias 0 -> 1
- net unconnected-(U1-NC-Pad1): track 0.00 -> 9.15 mm
- net unconnected-(D3-K-Pad1): track 0.00 -> 9.13 mm
- net unconnected-(R10-Pad1): track 0.00 -> 8.54 mm, vias 0 -> 1
- net unconnected-(U3-Q7-Pad9): track 0.00 -> 8.39 mm
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Other:
- outline, holes or cut-outs redrawn

Commit message: loin
Parts:
- added C12: C_Polarized, Capacitor_THT:CP_Radial_D5.0mm_P2.00mm, F.Cu at (165.9, 123.3)
- added Q1: 2N3904, Package_TO_SOT_THT:TO-92, F.Cu at (130.7, 123.6)
- added R19: 270 Ω ±5%, Resistor_THT:R_Axial_DIN0207_L6.3mm_D2.5mm_P10.16mm_Horizontal, F.Cu at (130.7, 118.6)
- added R20: 100 kΩ ±5%, Resistor_THT:R_Axial_DIN0207_L6.3mm_D2.5mm_P10.16mm_Horizontal, F.Cu at (137.2, 121.5)
- added R21: 100 kΩ ±5%, Resistor_THT:R_Axial_DIN0207_L6.3mm_D2.5mm_P10.16mm_Horizontal, F.Cu at (143.5, 118.6)
- added R22: 100 kΩ ±5%, Resistor_THT:R_Axial_DIN0207_L6.3mm_D2.5mm_P10.16mm_Horizontal, F.Cu at (149.9, 121.7)
- added R23: 100 Ω ±1%, Resistor_THT:R_Axial_DIN0207_L6.3mm_D2.5mm_P10.16mm_Horizontal, F.Cu at (156.3, 118.6)
- moved C7 7.56 mm to (146.1, 123.9), turned to -90 degrees
- moved C2 0.73 mm to (116.5, 112.3)
- moved C1 0.59 mm to (116.5, 105.4)
- moved R3 0.53 mm to (117.9, 118.7)
- moved R4 0.34 mm to (117.9, 121.8)
- moved R6 0.29 mm to (117.7, 131.6)
Connections:
- C1 pad 1: unconnected-(C1-Pad1) -> VCC
- C2 pad 1: unconnected-(C2-Pad1) -> VCC
- D1 pad 1: unconnected-(D1-K-Pad1) -> VCC
- D1 pad 2: unconnected-(D1-A-Pad2) -> Net-(D1-A)
- D3 pad 1: unconnected-(D3-K-Pad1) -> Net-(D3-K)
- J1 pad 1: unconnected-(J1-Pin_1-Pad1) -> GND
- J1 pad 14: unconnected-(J1-Pin_14-Pad14) -> Net-(J1-Pin_14)
- J1 pad 7: unconnected-(J1-Pin_7-Pad7) -> D3
- J1 pad 9: unconnected-(J1-Pin_9-Pad9) -> D1
- R1 pad 2: unconnected-(R1-Pad2) -> Net-(J1-Pin_14)
- R3 pad 1: unconnected-(R3-Pad1) -> GND
- R4 pad 1: unconnected-(R4-Pad1) -> VCC
- R5 pad 2: unconnected-(R5-Pad2) -> Net-(Q1-B)
- R6 pad 2: Net-(U5-SwC) -> Net-(D1-A)
- U4 pad 13: unconnected-(U4-Pad13) -> Net-(U4-Pad13)
- U4 pad 3: unconnected-(U4-Pad3) -> Net-(U4-Pad13)
- U5 pad 1: Net-(U5-SwC) -> Net-(D1-A)
- U5 pad 2: unconnected-(U5-SwE-Pad2) -> GND
- U5 pad 7: unconnected-(U5-Ipk-Pad7) -> Net-(Q1-C)
- U6 pad 2: unconnected-(U6-A12-Pad2) -> Net-(U6-A12)
- U6 pad 26: unconnected-(U6-A13-Pad26) -> Net-(U6-A12)
Routing:
- net Net-(U6-A12): track 0.00 -> 27.3 mm, vias 0 -> 1
- net unconnected-(J1-Pin_4-Pad4): track 0.00 -> 25.5 mm, vias 0 -> 1
- net unconnected-(J1-Pin_3-Pad3): track 0.00 -> 20.9 mm, vias 0 -> 1
- net Net-(D1-A): track 0.00 -> 20.5 mm, vias 0 -> 1
- net unconnected-(D1-A-Pad2): track 17.9 -> 0.00 mm, vias 1 -> 0
- net D3: track 45.1 -> 61.4 mm
- net Net-(U5-Vin): track 0.00 -> 16.2 mm, vias 0 -> 1
- net Net-(Q1-C): track 0.00 -> 16.0 mm
- net unconnected-(U6-~{PGM}-Pad27): track 0.00 -> 13.9 mm, vias 0 -> 1
- net unconnected-(U6-A11-Pad23): track 0.00 -> 12.7 mm, vias 0 -> 1
- net unconnected-(U6-A9-Pad24): track 0.00 -> 12.7 mm, vias 0 -> 1
- net unconnected-(U6-A8-Pad25): track 0.00 -> 12.7 mm, vias 0 -> 1
- net Net-(D3-K): track 0.00 -> 9.69 mm, vias 0 -> 1
- net unconnected-(U6-A0-Pad10): track 0.00 -> 9.13 mm
- net unconnected-(D3-K-Pad1): track 9.13 -> 0.00 mm
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