File: servicetastatur.kicad_sch (KiCad schematic)
At the start: 7 parts, among them U1 AT24CS16-SSHM, U2 TL7705A, U3 74HC165, U4 74HC00, U5 MC34063AP, U6 27C128, Y1 Crystal

Commit message: kleiner
Parts:
- added C1, C2: C_Polarized, Capacitor_THT:CP_Radial_D5.0mm_P2.00mm, symbol Device:C_Polarized
- added J1: Conn_01x16_Socket, Connector_JST:JST_ZE_B16B-ZESK-1D_1x16_P1.50mm_Vertical, symbol Connector:Conn_01x16_Socket
- added J2: Conn_01x06_Socket, Connector_Hirose:Hirose_DF63-6P-3.96DSA_1x06_P3.96mm_Vertical, symbol Connector:Conn_01x06_Socket
Changed lines of the file:
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@@
+    )
+  )
+  (symbol (lib_id "Device:C_Polarized") (at 68.58 101.6 0) (unit 1)
+    (in_bom yes) (on_board yes) (dnp no) (fields_autoplaced)
+    (property "Reference" "C1" (at 72.39 99.441 0)
+      (effects (font (size 1.27 1.27)) (justify left))
+    )
+    (property "Value" "C_Polarized" (at 72.39 101.981 0)
+      (effects (font (size 1.27 1.27)) (justify left))
+    )
+    (property "Footprint" "Capacitor_THT:CP_Radial_D5.0mm_P2.00mm" (at 69.5452 105.41 0)
+      (effects (font (size 1.27 1.27)) hide)
+    )
+    (property "Datasheet" "~" (at 68.58 101.6 0)
+      (effects (font (size 1.27 1.27)) hide)
+    )
+    (pin "1")
+    (pin "2")
+    (instances
+      (project "servicetastatur"
+        (path "/f1547e98-e012-47b0-8f5e-c4ff3a098fc5"
+          (reference "C1") (unit 1)
+        )
+      )
     )
   )
@@
     )
   )
+  (symbol (lib_id "Device:C_Polarized") (at 87.63 101.6 0) (unit 1)
+    (in_bom yes) (on_board yes) (dnp no) (fields_autoplaced)
+    (property "Reference" "C2" (at 91.44 99.441 0)
+      (effects (font (size 1.27 1.27)) (justify left))
+    )
+    (property "Value" "C_Polarized" (at 91.44 101.981 0)
+      (effects (font (size 1.27 1.27)) (justify left))
+    )
+    (property "Footprint" "Capacitor_THT:CP_Radial_D5.0mm_P2.00mm" (at 88.5952 105.41 0)
+      (effects (font (size 1.27 1.27)) hide)
+    )
+    (property "Datasheet" "~" (at 87.63 101.6 0)
+      (effects (font (size 1.27 1.27)) hide)
+    )
+    (pin "1")
+    (pin "2")
+    (instances
+      (project "servicetastatur"
+        (path "/f1547e98-e012-47b0-8f5e-c4ff3a098fc5"
+          (reference "C2") (unit 1)
+        )
+      )
+    )
+  )
   (symbol (lib_id "Memory_EEPROM:AT24CS16-SSHM") (at 160.02 90.17 0) (unit 1)
     (in_bom yes) (on_board yes) (dnp no) (fields_autoplaced)
@@
     )
   )
+  (symbol (lib_id "Connector:Conn_01x16_Socket") (at 36.83 52.07 0) (unit 1)
+    (in_bom yes) (on_board yes) (dnp no) (fields_autoplaced)
+    (property "Reference" "J1" (at 38.1 52.07 0)
+      (effects (font (size 1.27 1.27)) (justify left))
+    )
+    (property "Value" "Conn_01x16_Socket" (at 38.1 54.61 0)
+      (effects (font (size 1.27 1.27)) (justify left))
+    )
+    (property "Footprint" "Connector_JST:JST_ZE_B16B-ZESK-1D_1x16_P1.50mm_Vertical" (at 36.83 52.07 0)
+      (effects (font (size 1.27 1.27)) hide)
+    )
+    (property "Datasheet" "~" (at 36.83 52.07 0)
+      (effects (font (size 1.27 1.27)) hide)
+    )
+    (pin "1")
+    (pin "10")
+    (pin "11")
+    (pin "12")
+    (pin "13")
+    (pin "14")
+    (pin "15")
+    (pin "16")
+    (pin "2")
+    (pin "3")
+    (pin "4")
+    (pin "5")
+    (pin "6")
+    (pin "7")
+    (pin "8")
+    (pin "9")
+    (instances
+      (project "servicetastatur"
+        (path "/f1547e98-e012-47b0-8f5e-c4ff3a098fc5"
+          (reference "J1") (unit 1)
+        )
+      )
+    )
+  )
   (symbol (lib_id "Regulator_Switching:MC34063AP") (at 88.9 168.91 0) (unit 1)
     (in_bom yes) (on_board yes) (dnp no) (fields_autoplaced)
@@
         )
       )
+    )
+  )
+  (symbol (lib_id "Connector:Conn_01x06_Socket") (at 148.59 39.37 0) (unit 1)
+    (in_bom yes) (on_board yes) (dnp no) (fields_autoplaced)
+    (property "Reference" "J2" (at 149.86 39.37 0)
+      (effects (font (size 1.27 1.27)) (justify left))
+    )
+    (property "Value" "Conn_01x06_Socket" (at 149.86 41.91 0)
+      (effects (font (size 1.27 1.27)) (justify left))
+    )
+    (property "Footprint" "Connector_Hirose:Hirose_DF63-6P-3.96DSA_1x06_P3.96mm_Vertical" (at 148.59 39.37 0)
+      (effects (font (size 1.27 1.27)) hide)
+    )
+    (property "Datasheet" "~" (at 148.59 39.37 0)
+      (effects (font (size 1.27 1.27)) hide)
+    )
+    (pin "1")
+    (pin "2")
+    (pin "3")
+    (pin "4")
+    (pin "5")
+    (pin "6")
+    (instances
+      (project "servicetastatur"
+        (path "/f1547e98-e012-47b0-8f5e-c4ff3a098fc5"
+          (reference "J2") (unit 1)
+        )
+      )

Commit message: rumgeschiebe
Parts:
- J2: footprint Connector_Hirose:Hirose_DF63-6P-3.96DSA_1x06_P3.96mm_Vertical -> Connector_JST:JST_PH_S6B-PH-K_1x06_P2.00mm_Horizontal
Changed lines of the file:
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@@
       (effects (font (size 1.27 1.27)) (justify left))
     )
-    (property "Footprint" "Connector_Hirose:Hirose_DF63-6P-3.96DSA_1x06_P3.96mm_Vertical" (at 148.59 39.37 0)
+    (property "Footprint" "Connector_JST:JST_PH_S6B-PH-K_1x06_P2.00mm_Horizontal" (at 148.59 39.37 0)
       (effects (font (size 1.27 1.27)) hide)
     )

Commit message: anschluss
Parts:
- J1: footprint Connector_JST:JST_ZE_B16B-ZESK-1D_1x16_P1.50mm_Vertical -> Connector_Molex:Molex_Picoflex_90325-0016_2x08_P1.27mm_Vertical
- J2: footprint Connector_JST:JST_PH_S6B-PH-K_1x06_P2.00mm_Horizontal -> Connector_Molex:Molex_SPOX_5268-06A_1x06_P2.50mm_Horizontal
Changed lines of the file:
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@@
       (effects (font (size 1.27 1.27)) (justify left))
     )
-    (property "Footprint" "Connector_JST:JST_ZE_B16B-ZESK-1D_1x16_P1.50mm_Vertical" (at 36.83 52.07 0)
+    (property "Footprint" "Connector_Molex:Molex_Picoflex_90325-0016_2x08_P1.27mm_Vertical" (at 36.83 52.07 0)
       (effects (font (size 1.27 1.27)) hide)
     )
@@
       (effects (font (size 1.27 1.27)) (justify left))
     )
-    (property "Footprint" "Connector_JST:JST_PH_S6B-PH-K_1x06_P2.00mm_Horizontal" (at 148.59 39.37 0)
+    (property "Footprint" "Connector_Molex:Molex_SPOX_5268-06A_1x06_P2.50mm_Horizontal" (at 148.59 39.37 0)
       (effects (font (size 1.27 1.27)) hide)
     )

Commit message: i mag ned mehr
Parts:
- J2: footprint Connector_Molex:Molex_SPOX_5268-06A_1x06_P2.50mm_Horizontal -> Connector_Molex:Molex_Nano-Fit_105313-xx06_1x06_P2.50mm_Horizontal
Changed lines of the file:
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@@
       (effects (font (size 1.27 1.27)) (justify left))
     )
-    (property "Footprint" "Connector_Molex:Molex_SPOX_5268-06A_1x06_P2.50mm_Horizontal" (at 148.59 39.37 0)
+    (property "Footprint" "Connector_Molex:Molex_Nano-Fit_105313-xx06_1x06_P2.50mm_Horizontal" (at 148.59 39.37 0)
       (effects (font (size 1.27 1.27)) hide)
     )

Commit message: sdfsdf
Parts:
- removed J1: Conn_01x16_Socket, Connector_Molex:Molex_Picoflex_90325-0016_2x08_P1.27mm_Vertical, symbol Connector:Conn_01x16_Socket
- added C3, C4, C5, C6, C7: C, Capacitor_THT:C_Axial_L3.8mm_D2.6mm_P7.50mm_Horizontal, symbol Device:C
- added J1: Conn_02x08_Odd_Even, Connector_PinSocket_1.00mm:PinSocket_1x16_P1.00mm_Vertical_SMD_Pin1Right, symbol Connector_Generic:Conn_02x08_Odd_Even
- added R1, R4: 3.3 kΩ ±5%, Resistor_THT:R_Axial_DIN0207_L6.3mm_D2.5mm_P10.16mm_Horizontal, symbol Device:R
- added R2: 22 Ω ±5%, Resistor_THT:R_Axial_DIN0207_L6.3mm_D2.5mm_P10.16mm_Horizontal, symbol Device:R
- added R3: 110 Ω ±1%, Resistor_THT:R_Axial_DIN0207_L6.3mm_D2.5mm_P10.16mm_Horizontal, symbol Device:R
- added R5: 270 Ω ±5%, Resistor_THT:R_Axial_DIN0207_L6.3mm_D2.5mm_P10.16mm_Horizontal, symbol Device:R
Connections:
- net GND: now reaches U6.14 (GND)
- net GND: now also U1.4 (GND), U2.4 (GND), U3.8 (GND), U4.7 (GND), U5.4 (GND), C3.1, C4.1, C5.1, C6.1, C7.1, R1.1
- net at U1.8 (VCC): now also C5.2
- net at U3.16 (VCC): now also C3.2
- net at U2.8 (VCC): now also C6.2
- net at U5.6 (Vin): now also C7.2
- net at U4.14 (VCC): now also C4.2

Commit message: CPU
Parts:
- added C8, C9: C, Capacitor_THT:CP_Radial_Tantal_D4.5mm_P2.50mm, symbol Device:C
- added D1, D2: D, Diode_THT:D_DO-15_P15.24mm_Horizontal, symbol Device:D
- added R6: R, Resistor_THT:R_Axial_DIN0414_L11.9mm_D4.5mm_P15.24mm_Horizontal, symbol Device:R
- added U7: ~, Package_LCC:PLCC-44_THT-Socket, symbol MCU_Atmel:TS80C31
Connections:
- net GND: now also C1.2, C2.2, U4.12, D2.2 (A), U7.1 (Vss1), U7.22 (Vss); no longer C6.1
- net at U4.10: now also U7.18 (P3.6/WR)
- net at U4.9: now also U7.19 (P3.7/RD)
- net VCC: now reaches C4.2, U4.14 (VCC)
- net VCC: now also C3.2, U3.16 (VCC), U6.28 (VCC), U7.44 (Vcc)
- net at R4.2: now also R3.2
- net D0: now reaches U6.11 (D0)
- net D0: now also U3.11 (D0), U7.43 (P0.0/AD0)
- net D1: now reaches U6.12 (D1)
- net D1: now also U3.12 (D1), U7.42 (P0.1/AD1)
- net D2: now reaches U6.13 (D2)
- net D2: now also U3.13 (D2), U7.41 (P0.2/AD2)
- net D3: now reaches U6.15 (D3)
- net D3: now also U3.14 (D3), U7.40 (P0.3/AD3)
- net D4: now reaches U6.16 (D4)
- net D4: now also U3.3 (D4), U7.39 (P.04/AD4)
- net D5: now reaches U6.17 (D5)
- net D5: now also U3.4 (D5), U7.38 (P0.5/AD5)
- net D6: now reaches U6.18 (D6)
- net D6: now also U3.5 (D6), U7.37 (P0.6/AD6)
- net D7: now reaches U6.19 (D7)
- net D7: now also U3.6 (D7), U7.36 (P0.7/AD7)
- net at U6.20 (~{CE}): now also U7.32 (PSEN)
- net at Y1.1: now also C9.2, U7.21 (XTAL1)
- net at Y1.2: now also C8.2, U7.20 (XTAL2)
- net at U4.11: now also U7.14 (P3.2/INT0)
- net at U1.7 (WP): now also C6.1
- net at U2.1 (REF): now also C6.2
- net at U2.8 (VCC): no longer C6.2
- net at U5.1 (SwC): now also R6.2
- new net: D2.1 (K), R6.1
- new net: C8.1, C9.1
Other:
- moved on the sheet: C5, C6, U1, U2, U4B, U4C, U4D, U6, Y1

Commit message: anschluss
Parts:
- added C10, C11: C, Capacitor_THT:CP_Radial_Tantal_D4.5mm_P2.50mm, symbol Device:C
- added D3: D, Diode_THT:D_DO-15_P15.24mm_Horizontal, symbol Device:D
- added J3: Conn_01x06, ConnPad:Conn01x06, symbol Connector_Generic:Conn_01x06
- added J4: Conn_01x02, symbol Connector_Generic:Conn_01x02
- added R10, R14, R7, R8, R9: 1 kΩ ±1%, Resistor_THT:R_Axial_DIN0207_L6.3mm_D2.5mm_P10.16mm_Horizontal, symbol Device:R
- added R11: 10 kΩ ±5%, Resistor_THT:R_Axial_DIN0207_L6.3mm_D2.5mm_P10.16mm_Horizontal, symbol Device:R
- added R12: 22 Ω ±5%, Resistor_THT:R_Axial_DIN0207_L6.3mm_D2.5mm_P10.16mm_Horizontal, symbol Device:R
- added R13: 47 kΩ ±5%, Resistor_THT:R_Axial_DIN0207_L6.3mm_D2.5mm_P10.16mm_Horizontal, symbol Device:R
- added R15: 4.7 kΩ ±1%, Resistor_THT:R_Axial_DIN0207_L6.3mm_D2.5mm_P10.16mm_Horizontal, symbol Device:R
- added R16: 47 Ω ±1%, Resistor_THT:R_Axial_DIN0207_L6.3mm_D2.5mm_P10.16mm_Horizontal, symbol Device:R
- added R17, R18: 270 Ω ±5%, Resistor_THT:R_Axial_DIN0207_L6.3mm_D2.5mm_P10.16mm_Horizontal, symbol Device:R
Connections:
- net GND: now also C6.1, U1.7 (WP), C10.1, R13.2
- net at U2.2 (~{RESIN}): now also R11.1
- net at U2.7 (SENSE): now also U2.8 (VCC), C11.1
- new net: R11.2, R7.1, R8.1, R9.1
- new net: J3.4 (Pin_4), R17.2, R8.2
- new net: J3.5 (Pin_5), R18.2, R7.2
- new net: J3.3 (Pin_3), R10.2, R9.2
- new net: C11.2, R12.2, R13.1
- new net: J3.2 (Pin_2), R16.2
- new net: D3.2 (A), J3.6 (Pin_6)
Other:
- moved on the sheet: C5, C6, U1, U2

Commit message: loin
Parts:
- added C12: C_Polarized, Capacitor_THT:CP_Radial_D5.0mm_P2.00mm, symbol Device:C_Polarized
- added Q1: 2N3904, Package_TO_SOT_THT:TO-92, symbol Transistor_BJT:2N3904
- added R19: 270 Ω ±5%, Resistor_THT:R_Axial_DIN0207_L6.3mm_D2.5mm_P10.16mm_Horizontal, symbol Device:R
- added R20, R21, R22: 100 kΩ ±5%, Resistor_THT:R_Axial_DIN0207_L6.3mm_D2.5mm_P10.16mm_Horizontal, symbol Device:R
- added R23: 100 Ω ±1%, Resistor_THT:R_Axial_DIN0207_L6.3mm_D2.5mm_P10.16mm_Horizontal, symbol Device:R
Connections:
- net D1: now also J1.9 (Pin_9)
- net D3: now also J1.7 (Pin_7)
- net GND: now also J1.1 (Pin_1), R3.1, U5.2 (SwE), C12.2
- net VCC: now also C1.1, C2.1, D1.1 (K), R4.1
- net at U4.3: now also U4.13
- net at U6.2 (A12): now also U6.26 (A13)
- net at R6.2, U5.1 (SwC): now also D1.2 (A)
- net at R5.2: now also Q1.2 (B), R19.1
- net at U5.7 (Ipk): now also Q1.3 (C), R20.1, R21.1
- net at R1.2: now also J1.14 (Pin_14)
- net at D3.1 (K): now also R23.2
- new net: R20.2, R21.2, R22.1
Other:
- moved on the sheet: C7, D1, D2, J4, R1, R2, R3, R4, R5, R6, U4A, U4B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
