File: servicetastatur.kicad_sch (KiCad schematic)
At the start: 51 parts, among them J1 Conn_02x08_Odd_Even, J2 Conn_01x06_Socket, J3 Conn_01x06, J4 Conn_01x02, Q1 2N3904, U1 AT24CS16-SSHM, U2 TL7705A, U3 74HC165, U4 74HC00, U5 MC34063AP, U6 27C128, Y1 Crystal

Commit message: 2024 update
Parts:
- added C13, C14, C15, C16, C17, C18: C, Capacitor_THT:C_Axial_L3.8mm_D2.6mm_P7.50mm_Horizontal, symbol Device:C
- added C19, C20, C21: C, Capacitor_THT:CP_Radial_Tantal_D4.5mm_P2.50mm, symbol Device:C
- added D4: D, Diode_THT:D_A-405_P7.62mm_Horizontal, symbol Device:D
- added R24, R26, R27: 100 kΩ ±5%, Resistor_THT:R_Axial_DIN0207_L6.3mm_D2.5mm_P10.16mm_Horizontal, symbol Device:R
- added R25: 4.7 kΩ ±1%, Resistor_THT:R_Axial_DIN0207_L6.3mm_D2.5mm_P10.16mm_Horizontal, symbol Device:R
- added U1: 74HC238, Package_DIP:DIP-16_W7.62mm, symbol 74xx:74HC238
- added U5: 74LS573, Package_DIP:DIP-20_W7.62mm, symbol 74xx:74LS573
- J1: renamed from J4; footprint (none) -> Connector_Wire:SolderWire-0.5sqmm_1x02_P4.8mm_D0.9mm_OD2.3mm
- J2: renamed from J1; value Conn_02x08_Odd_Even -> LCD; footprint Connector_PinSocket_1.00mm:PinSocket_1x16_P1.00mm_Vertical_SMD_Pin1Right -> (none)
- J3: value Conn_01x06 -> Automat
- J4: renamed from J2; value Conn_01x06_Socket -> Tasten
- renumbered U5 to U18, U4 to U2, U6 to U3, U7 to U4, U2 to U7, U3 to U8, U1 to U9
Connections:
- net D0: now also U5.9 (D7)
- net D1: now also U5.8 (D6)
- net D2: now also U5.7 (D5)
- net D3: now also U5.6 (D4)
- net D4: now also U5.5 (D3)
- net D5: now also U5.4 (D2)
- net D6: now also U5.3 (D1)
- net D7: now also U5.2 (D0)
- net GND: now also U4.35 (EA), C13.1, C14.2, C15.1, C16.1, C18.1, C19.2, C20.2, C21.2, U1.8 (GND), U5.1 (OE), U5.10 (GND)
- net VCC: now also C11.1, R11.2, R7.1, R8.1, R9.1, U7.7 (SENSE), U7.8 (VCC), C18.2, R25.1, U5.20 (VCC)
- net at U2.4: now also U2.5
- net at U4.24 (P2.0/A8): now also U3.25 (A8)
- net at U4.25 (P2.1/A9): now also U3.24 (A9)
- net at U4.26 (P2.2/A10): now also U3.21 (A10)
- net at U4.27 (P2.3/A11): now also U3.23 (A11)
- net at U4.28 (P2.4/A12): now also U3.2 (A12)
- net at U4.29 (P2.5/A13): now also U3.26 (A13)
- net A14: now reaches U4.30 (P2.6/A14)
- net A14: now also U1.4 (~{E1})
- net A15: now reaches U4.31 (P2.7/A15)
- net A15: now also R24.2, U1.5 (~{E2})
- net ALE: now reaches U4.33 (ALE)
- net ALE: now also U5.11 (Load)
- net at U3.10 (A0): now also U5.12 (Q7)
- net at U3.3 (A7): now also U5.19 (Q0)
- net at U3.4 (A6): now also U5.18 (Q1)
- net at U3.5 (A5): now also U5.17 (Q2)
- net at U3.6 (A4): now also U5.16 (Q3)
- net at U3.7 (A3): now also U5.15 (Q4)
- net at U3.8 (A2): now also U5.14 (Q5)
- net at U3.9 (A1): now also U5.13 (Q6)
- net at J1.1 (Pin_1): now also R27.2
- net at J1.2 (Pin_2): now also R26.2
- net at U8.10 (DS): now also R14.1, U8.15 (~{CE})
- net at U7.6 (RESET): now also R12.1
- net at C12.1: now also R22.2
- new net: R24.1, R25.2
- no-connect marks 0 -> 4
Other:
- moved on the sheet: C12, C3, C7, D1, D2, J1, Q1, R14, R20, R21, R22, R3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

Commit message: caps
Connections:
- net VCC: now also C14.1, C20.1
Changed lines of the file:
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@@
+	)
+	(symbol
+		(lib_id "power:VCC")
+		(at 295.91 168.91 270)
+		(unit 1)
+		(exclude_from_sim no)
+		(in_bom yes)
+		(on_board yes)
+		(dnp no)
+		(fields_autoplaced yes)
+		(property "Reference" "#PWR051"
+			(at 292.1 168.91 0)
+			(effects
+				(font
+					(size 1.27 1.27)
+				)
+				(hide yes)
+			)
+		)
+		(property "Value" "VCC"
+			(at 299.72 168.9099 90)
+			(effects
+				(font
+					(size 1.27 1.27)
+				)
+				(justify left)
+			)
+		)
+		(property "Footprint" ""
+			(at 295.91 168.91 0)
+			(effects
+				(font
+					(size 1.27 1.27)
+				)
+				(hide yes)
+			)
+		)
+		(property "Datasheet" ""
+			(at 295.91 168.91 0)
+			(effects
+				(font
+					(size 1.27 1.27)
+				)
+				(hide yes)
+			)
+		)
+		(property "Description" ""
+			(at 295.91 168.91 0)
+			(effects
+				(font
+					(size 1.27 1.27)
+				)
+				(hide yes)
+			)
+		)
+		(pin "1"
+		)
+		(instances
+			(project "servicetastatur"
+				(path "/f1547e98-e012-47b0-8f5e-c4ff3a098fc5"
+					(reference "#PWR051")
+					(unit 1)
+				)
+			)
+		)
 	)
 	(symbol
@@
 					(unit 1)
 				)
+			)
+		)
+	)
+	(symbol
+		(lib_id "power:VCC")
+		(at 252.73 184.15 0)
+		(unit 1)
+		(exclude_from_sim no)
+		(in_bom yes)
+		(on_board yes)
+		(dnp no)
+		(fields_autoplaced yes)
+		(property "Reference" "#PWR050"
+			(at 252.73 187.96 0)
+			(effects
+				(font
+					(size 1.27 1.27)
+				)
+				(hide yes)
+			)
+		)
+		(property "Value" "VCC"
+			(at 252.73 179.07 0)
+			(effects
+				(font
+					(size 1.27 1.27)
+				)
+			)
+		)
+		(property "Footprint" ""
+			(at 252.73 184.15 0)
+			(effects
+				(font
+					(size 1.27 1.27)
+				)
+				(hide yes)
+			)
+		)
+		(property "Datasheet" ""
+			(at 252.73 184.15 0)
+			(effects
+				(font
+					(size 1.27 1.27)
+				)
+				(hide yes)
+			)
+		)
+		(property "Description" ""
+			(at 252.73 184.15 0)
+			(effects
+				(font
+					(size 1.27 1.27)
+				)
+				(hide yes)
+			)
+		)
+		(pin "1"
+		)
+		(instances
+			(project "servicetastatur"
+				(path "/f1547e98-e012-47b0-8f5e-c4ff3a098fc5"
+					(reference "#PWR050")
+					(unit 1)
+				)

Commit message: shift register
Parts:
- added U6, U7: 74HC4094, Package_DIP:DIP-16_W7.62mm, symbol MCU_Atmel:74HC4094
- J2: footprint (none) -> Connector_TE-Connectivity:TE_Micro-MaTch_1-215079-6_2x08_P1.27mm_Vertical
- renumbered U7 to U17
Connections:
- net D0: now also U6.11 (QP7), U7.11 (QP7)
- net D1: now also U6.14 (QP4), U7.12 (QP6)
- net D2: now also U6.13 (QP5), U7.13 (QP5)
- net D3: now also U6.12 (QP6), U7.14 (QP4)
- net D4: now also U6.7 (QP3), U7.7 (QP3)
- net D5: now also U6.6 (QP2), U7.6 (QP2)
- net D6: now also U6.5 (QP1), U7.5 (QP1)
- net D7: now also U6.4 (QP0), U7.4 (QP0)
- net GND: now also C17.1, R14.2, U6.8 (GND), U7.8 (GND)
- net VCC: now also C15.2, C16.2, C17.2, U1.16 (VCC), U6.16 (VCC), U7.16 (VCC)
- net at U2.4, U2.5: now also U1.9 (Y6)
- net at U2.6: now also U8.1 (~{PL})
- net RESET: now reaches U4.10 (RST)
- net SDA: now reaches U4.16 (P3.4/T0)
- net SDA: now also U9.5 (SDA)
- net SCL: now reaches U4.17 (P3.5/T1)
- net SCL: now also U9.6 (SCL)
- net at U4.2 (P1.0): now also J4.1 (Pin_1)
- net at U4.3 (P1.1): now also J4.2 (Pin_2)
- net at U3.20 (~{CE}), U4.32 (PSEN): now also U3.22 (~{OE})
- net at U4.4 (P1.2): now also J4.3 (Pin_3)
- net at U2.1: now also U2.2
- net at U8.9 (Q7): now also R16.1
- net at U1.10 (Y5): now also U6.15 (OE)
- net at U1.11 (Y4): now also U7.15 (OE)
- new net: U6.2 (D), U7.9 (QS1)
- new net: U6.3 (CP), U7.3 (CP)
- no-connect marks 4 -> 9
Other:
- moved on the sheet: C1, C13, C14, C15, C16, C17, C2, C3, C4, D3, D4, J1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

Commit message: stecker
Parts:
- added C22: C, Capacitor_THT:C_Axial_L3.8mm_D2.6mm_P7.50mm_Horizontal, symbol Device:C
- J2: footprint Connector_TE-Connectivity:TE_Micro-MaTch_1-215079-6_2x08_P1.27mm_Vertical -> adp:FFC_2x08_P1mm_Vertical
- J4: footprint Connector_Molex:Molex_Nano-Fit_105313-xx06_1x06_P2.50mm_Horizontal -> adp:FFC_1x06_P2.50mm_Horizontal
- U9: symbol Memory_EEPROM:AT24CS16-SSHM -> Memory_EEPROM:24LC16
- Y1: value Crystal -> 11.059
Connections:
- net A14: now also U3.27 (~{PGM})
- net A15: now also U3.1 (VPP), U4.34 (NIC)
- net D2: now also J2.8 (Pin_8)
- net D5: now also J2.5 (Pin_5)
- net GND: now also C8.1, C9.1, D4.2 (A), J3.1 (Pin_1), R15.2, U9.1 (A0), U9.2 (A1), U9.3 (A2), C22.1; no longer C13.1, D2.2 (A), R1.1, U18.2 (SwE), U2.12
- net VCC: now also C21.1, C5.2, J2.15 (Pin_15), U9.8 (VCC), C22.2; no longer D1.1 (K)
- net at U4.15 (P3.3/INT1): now also U2.12, U2.13, U2.3
- net at U4.6 (P1.4): now also J4.4 (Pin_4)
- net at U4.7 (P1.5): now also J4.5 (Pin_5)
- net at U4.8 (P1.6): now also J4.6 (Pin_6)
- net at R18.1: now also U7.2 (D)
- net at U2.8: now also U1.6 (E3)
- net at R20.2, R21.2, R22.1: now also C7.2, D3.1 (K), R23.2, U18.6 (Vin)
- net at U3.9 (A1), U5.13 (Q6): now also J2.13 (Pin_13)
- net at D2.1 (K), R6.1: now also Q1.1 (E)
- net at R3.2, R4.2: now also U18.5 (Vfb)
- net at R2.2: now also J2.2 (Pin_2)
- net at U2.1, U2.2: now also R10.1
- net CLOCK: now reaches R17.1
- net CLOCK: now also U6.3 (CP), U7.3 (CP), U8.2 (CP)
- net at R19.2: now also U18.8 (DC)
- net at D4.1 (K): now also C13.1, R15.1
- net at U6.1 (STR): now also U7.1 (STR)
- net at C19.1: now also R22.2
- net at R23.1: now also C12.1
- no-connect marks 9 -> 14
Other:
- moved on the sheet: C1, C10, C11, C12, C13, C14, C15, C16, C17, C18, C19, C2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

Commit message: spekulation
Connections:
- net RESET: now also C11.2, R12.2, R13.1
- net VCC: now also D1.1 (K)
- net at U3.6 (A4), U5.16 (Q3): now also U1.1 (A0)
- net at U3.5 (A5), U5.17 (Q2): now also U1.2 (A1)
- net at U3.4 (A6), U5.18 (Q1): now also U1.3 (A2)
Changed lines of the file:
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@@
 	)
 	(junction
+		(at 283.21 45.72)
+		(diameter 0)
+		(color 0 0 0 0)
+	)
+	(junction
 		(at 21.59 181.61)
 		(diameter 0)
@@
 	)
 	(junction
-		(at 191.77 83.82)
+		(at 280.67 50.8)
 		(diameter 0)
 		(color 0 0 0 0)
 	)
 	(junction
-		(at 187.96 297.18)
+		(at 191.77 83.82)
 		(diameter 0)
 		(color 0 0 0 0)
 	)
 	(junction
-		(at 280.67 38.1)
+		(at 187.96 297.18)
 		(diameter 0)
 		(color 0 0 0 0)
@@
 	)
 	(junction
+		(at 288.29 35.56)
+		(diameter 0)
+		(color 0 0 0 0)
+	)
+	(junction
 		(at 177.8 63.5)
 		(diameter 0)
@@
 	)
 	(junction
-		(at 241.3 251.46)
+		(at 285.75 38.1)
 		(diameter 0)
 		(color 0 0 0 0)
 	)
 	(junction
-		(at 283.21 35.56)
+		(at 241.3 251.46)
 		(diameter 0)
 		(color 0 0 0 0)
@@
 	)
 	(junction
+		(at 281.94 48.26)
+		(diameter 0)
+		(color 0 0 0 0)
+	)
+	(junction
 		(at 87.63 166.37)
 		(diameter 0)
@@
 	(wire
 		(pts
-			(xy 280.67 38.1) (xy 280.67 0)
+			(xy 285.75 38.1) (xy 285.75 0)
 		)
 		(stroke
@@
 	(wire
 		(pts
-			(xy -7.62 -2.54) (xy 283.21 -2.54)
+			(xy -7.62 -2.54) (xy 288.29 -2.54)
 		)
 		(stroke
@@
 	(wire
 		(pts
-			(xy 275.59 38.1) (xy 280.67 38.1)
+			(xy 275.59 38.1) (xy 285.75 38.1)
 		)
 		(stroke
@@
 	(wire
 		(pts
+			(xy 33.02 3.81) (xy 33.02 17.78)
+		)
+		(stroke
+			(width 0)
+			(type default)
+		)
+	)
+	(wire
+		(pts
 			(xy 125.73 27.94) (xy 125.73 30.48)
 		)
@@
 	(wire
 		(pts
+			(xy 31.75 5.08) (xy 31.75 20.32)
+		)
+		(stroke
+			(width 0)
+			(type default)
+		)
+	)
+	(wire
+		(pts
 			(xy 229.87 64.77) (xy 229.87 63.5)
 		)
@@
 	(wire
 		(pts
-			(xy 275.59 35.56) (xy 283.21 35.56)
+			(xy 275.59 35.56) (xy 288.29 35.56)
 		)
 		(stroke
@@
 	(wire
 		(pts
-			(xy 283.21 -2.54) (xy 283.21 35.56)
+			(xy 288.29 -2.54) (xy 288.29 35.56)
 		)
 		(stroke
@@
 	(wire
 		(pts
+			(xy 31.75 5.08) (xy 280.67 5.08)
+		)
+		(stroke
+			(width 0)
+			(type default)
+		)
+	)
+	(wire
+		(pts
 			(xy 60.96 27.94) (xy 54.61 27.94)
 		)
@@
 	(wire
 		(pts
+			(xy 34.29 15.24) (xy 34.29 2.54)
+		)
+		(stroke
+			(width 0)
+			(type default)
+		)
+	)
+	(wire
+		(pts
 			(xy 201.93 177.8) (xy 201.93 134.62)
 		)
@@
 	(wire
 		(pts
+			(xy 31.75 20.32) (xy 34.29 20.32)
+		)
+		(stroke
+			(width 0)
+			(type default)
+		)
+	)
+	(wire
+		(pts
 			(xy 95.25 92.71) (xy 104.14 92.71)
 		)
@@
 	(wire
 		(pts
+			(xy 34.29 2.54) (xy 283.21 2.54)
+		)
+		(stroke
+			(width 0)
+			(type default)
+		)
+	)
+	(wire
+		(pts
 			(xy 181.61 60.96) (xy 181.61 63.5)
 		)
@@
 	(wire
 		(pts
-			(xy 275.59 48.26) (xy 288.29 48.26)
+			(xy 275.59 48.26) (xy 281.94 48.26)
 		)
 		(stroke
@@
 	(wire
 		(pts
-			(xy 280.67 0) (xy -5.08 0)
+			(xy 285.75 0) (xy -5.08 0)
 		)
 		(stroke
@@
 	(wire
 		(pts
+			(xy 283.21 45.72) (xy 283.21 2.54)
+		)
+		(stroke
+			(width 0)
+			(type default)
+		)
+	)
+	(wire
+		(pts
 			(xy 198.12 45.72) (xy 198.12 43.18)
 		)
@@
 	(wire
 		(pts
-			(xy 95.25 102.87) (xy 104.14 102.87)
+			(xy 281.94 48.26) (xy 288.29 48.26)
 		)
 		(stroke
@@
 	(wire
 		(pts
-			(xy 227.33 177.8) (xy 201.93 177.8)
+			(xy 95.25 102.87) (xy 104.14 102.87)
 		)
 		(stroke
@@
 	(wire
 		(pts
-			(xy 229.87 66.04) (xy 288.29 66.04)
+			(xy 227.33 177.8) (xy 201.93 177.8)
 		)
 		(stroke
@@
 	(wire
 		(pts
-			(xy 283.21 35.56) (xy 288.29 35.56)
+			(xy 229.87 66.04) (xy 288.29 66.04)
 		)
 		(stroke
@@
 	(wire
 		(pts
+			(xy 285.75 38.1) (xy 288.29 38.1)
+		)
+		(stroke
+			(width 0)
+			(type default)
+		)
+	)
+	(wire
+		(pts
 			(xy 226.06 163.83) (xy 226.06 166.37)
 		)
@@
 	(wire
 		(pts
+			(xy 280.67 50.8) (xy 288.29 50.8)
+		)
+		(stroke
+			(width 0)
+			(type default)
+		)
+	)
+	(wire
+		(pts
 			(xy 240.03 163.83) (xy 241.3 163.83)
 		)
@@
 	(wire
 		(pts
+			(xy 283.21 45.72) (xy 288.29 45.72)
+		)
+		(stroke
+			(width 0)
+			(type default)
+		)
+	)
+	(wire
+		(pts
 			(xy 229.87 38.1) (xy 250.19 38.1)
 		)
@@
 	(wire
 		(pts
+			(xy 281.94 48.26) (xy 281.94 3.81)
+		)
+		(stroke
+			(width 0)
+			(type default)
+		)
+	)
+	(wire
+		(pts
 			(xy 195.58 48.26) (xy 195.58 45.72)
 		)
@@
 	(wire
 		(pts
-			(xy 275.59 45.72) (xy 288.29 45.72)
+			(xy 275.59 45.72) (xy 283.21 45.72)
 		)
 		(stroke
@@
 	(wire
 		(pts
-			(xy 280.67 38.1) (xy 288.29 38.1)
-		)
-		(stroke
-			(width 0)
-			(type default)
-		)
-	)
-	(wire
-		(pts
 			(xy 229.87 55.88) (xy 288.29 55.88)
 		)
@@
 	(wire
 		(pts
-			(xy 275.59 50.8) (xy 288.29 50.8)
+			(xy 275.59 50.8) (xy 280.67 50.8)
 		)
 		(stroke
@@
 	(wire
 		(pts
+			(xy 33.02 3.81) (xy 281.94 3.81)
+		)
+		(stroke
+			(width 0)
+			(type default)
+		)
+	)
+	(wire
+		(pts
 			(xy 100.33 100.33) (xy 100.33 95.25)
 		)
@@
 	(wire
 		(pts
+			(xy 280.67 50.8) (xy 280.67 5.08)
+		)
+		(stroke
+			(width 0)
+			(type default)
+		)
+	)
+	(wire
+		(pts
 			(xy 100.33 95.25) (xy 95.25 95.25)
 		)
@@
 	(wire
 		(pts
+			(xy 33.02 17.78) (xy 34.29 17.78)
+		)
+		(stroke
+			(width 0)
+			(type default)
+		)
+	)
+	(wire
+		(pts
 			(xy 95.25 90.17) (xy 104.14 90.17)
 		)
@@
 	(global_label "RESET"
 		(shape input)
-		(at 257.81 95.25 90)
+		(at 87.63 166.37 90)
 		(fields_autoplaced yes)
 		(effects
@@
 		)
 		(property "Intersheetrefs" "${INTERSHEET_REFS}"
-			(at 257.81 86.5197 90)
+			(at 87.63 157.6397 90)
 			(effects
 				(font
@@
 					(unit 1)
 				)
+			)
+		)
+	)
+	(symbol
+		(lib_id "power:VCC")
+		(at 201.93 273.05 180)
+		(unit 1)
+		(exclude_from_sim no)
+		(in_bom yes)
+		(on_board yes)
+		(dnp no)
+		(fields_autoplaced yes)
+		(property "Reference" "#PWR020"
+			(at 201.93 269.24 0)
+			(effects
+				(font
+					(size 1.27 1.27)
+				)
+				(hide yes)
+			)
+		)
+		(property "Value" "VCC"
+			(at 201.93 278.13 0)
+			(effects
+				(font
+					(size 1.27 1.27)
+				)
+			)
+		)
+		(property "Footprint" ""
+			(at 201.93 273.05 0)
+			(effects
+				(font
+					(size 1.27 1.27)
+				)
+				(hide yes)
+			)
+		)
+		(property "Datasheet" ""
+			(at 201.93 273.05 0)
+			(effects
+				(font
+					(size 1.27 1.27)
+				)
+				(hide yes)
+			)
+		)
+		(property "Description" ""
+			(at 201.93 273.05 0)
+			(effects
+				(font
+					(size 1.27 1.27)
+				)
+				(hide yes)
+			)
+		)
+		(pin "1"
+		)
+		(instances
+			(project "servicetastatur"
+				(path "/f1547e98-e012-47b0-8f5e-c4ff3a098fc5"
+					(reference "#PWR020")
+					(unit 1)
+				)

Commit message: layout
Parts:
- added R28, R29, R30: R, Resistor_THT:R_Axial_DIN0207_L6.3mm_D2.5mm_P10.16mm_Horizontal, symbol Device:R
- C1: footprint Capacitor_THT:CP_Radial_D5.0mm_P2.00mm -> Capacitor_THT:CP_Radial_D5.0mm_P2.50mm
- C3: renamed from C13; value C -> 68pF
- D1: footprint Diode_THT:D_DO-15_P15.24mm_Horizontal -> adp:D_DO-15_P15mm_Horizontal
- Q1: footprint Package_TO_SOT_THT:TO-92 -> adp:TO-92
- R15: renamed from R3; value 110 Ω ±1% -> 1 kΩ ±1%
- R26, R27: value 100 kΩ ±5% -> R
- R6: value R -> 220 Ω ±5%
- U4: value ~ -> 80C31
- U9: value AT24CS16-SSHM -> 24CS16
- renumbered C3 to C13, R15 to R3
Connections:
- net D0: now also J2.10 (Pin_10)
- net D4: now also J2.6 (Pin_6)
- net D6: now also J2.4 (Pin_4)
- net D7: now also J2.3 (Pin_3)
- net GND: now also D2.2 (A), J2.16 (Pin_16), J2.2 (Pin_2), R1.1, R2.2, U18.2 (SwE), R30.1
- net at C3.1, D4.1 (K), R3.1: now also U6.1 (STR), U7.1 (STR)
- net at C3.2: now also J3.3 (Pin_3), R10.2, R9.2
- net at Q1.3 (C), R20.1, R21.1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: now also R5.1
- net +VDC: now reaches D3.1 (K), R20.2, R21.2, R22.1, R23.2, U18.6 (Vin)
- net +VDC: no longer C7.2
- net A0: now reaches U3.10 (A0), U5.12 (Q7)
- net A0: now also J2.12 (Pin_12)
- net A1: now reaches J2.13 (Pin_13), U3.9 (A1), U5.13 (Q6)
- net A2: now reaches U3.8 (A2), U5.14 (Q5)
- net A3: now reaches U3.7 (A3), U5.15 (Q4)
- net A4: now reaches U1.1 (A0), U3.6 (A4), U5.16 (Q3)
- net A5: now reaches U1.2 (A1), U3.5 (A5), U5.17 (Q2)
- net A6: now reaches U1.3 (A2), U3.4 (A6), U5.18 (Q1)
- net A7: now reaches U3.3 (A7), U5.19 (Q0)
- net at C10.2: now also U17.3 (CT)
- net at U18.3 (TC): now also C7.2
- net at J2.11 (Pin_11): now also U1.7 (Y7)
- net at C12.1, R23.1: now also R28.1, R29.1
- no-connect marks 14 -> 19
Other:
- company: (none) -> https://github.com/stonedDiscord/servicetastatur
- title: (none) -> Blaue Servicetastatur
- moved on the sheet: C1, C10, C12, C13, C14, C15, C16, C17, C18, C19, C2, C20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

Commit message: so hab bestellt
Parts:
- removed R26, R27, R28, R29, R30: R, Resistor_THT:R_Axial_DIN0207_L6.3mm_D2.5mm_P10.16mm_Horizontal, symbol Device:R
- added J5, J6: Conn_01x03_Pin, Connector_PinSocket_2.54mm:PinSocket_1x03_P2.54mm_Vertical, symbol Connector:Conn_01x03_Pin
- R20, R21, R22: value 100 kΩ ±5% -> 1 Ω ±5%
Connections:
- net GND: now also J5.1 (Pin_1)
- net at J1.1 (Pin_1): now also J6.1 (Pin_1)
- net at J1.2 (Pin_2): now also J6.3 (Pin_3)
- net at C12.1, R23.1: now also J5.2 (Pin_2), J5.3 (Pin_3)
- no-connect marks 19 -> 15

Commit message: deko
Parts:
- D1, D3: value D -> 1N5819
- R1, R4: value 3.3 kΩ ±5% -> 3.3 kΩ
- R10, R14, R15, R7, R8, R9: value 1 kΩ ±1% -> 1 kΩ
- R11: value 10 kΩ ±5% -> 10 kΩ
- R12, R2: value 22 Ω ±5% -> 22 Ω
- R13: value 47 kΩ ±5% -> 47 kΩ
- R16: value 47 Ω ±1% -> 47 Ω
- R17, R18, R19, R5: value 270 Ω ±5% -> 270 Ω
- R20, R21, R22: value 1 Ω ±5% -> 1 Ω
- R23: value 100 Ω ±1% -> 100 Ω
- R24: value 100 kΩ ±5% -> 100 kΩ
- R25, R3: value 4.7 kΩ ±1% -> 4.7 kΩ
- R6: value 220 Ω ±5% -> 220 Ω
Changed lines of the file:
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@@
 			)
 		)
-		(property "Value" "1 kΩ ±1%"
+		(property "Value" "1 kΩ"
 			(at 229.87 163.195 90)
 			(effects
@@
 			)
 		)
-		(property "Value" "270 Ω ±5%"
+		(property "Value" "270 Ω"
 			(at 218.44 173.99 90)
 			(effects
@@
 			)
 		)
-		(property "Value" "1 Ω ±5%"
+		(property "Value" "1 Ω"
 			(at 318.77 181.61 90)
 			(effects
@@
 			)
 		)
-		(property "Value" "3.3 kΩ ±5%"
+		(property "Value" "3.3 kΩ"
 			(at 337.82 237.49 90)
 			(effects
@@
 			)
 		)
-		(property "Value" "22 Ω ±5%"
+		(property "Value" "22 Ω"
 			(at 34.29 138.43 90)
 			(effects
@@
 			)
 		)
-		(property "Value" "1 Ω ±5%"
+		(property "Value" "1 Ω"
 			(at 318.77 191.77 90)
 			(effects
@@
 			)
 		)
-		(property "Value" "270 Ω ±5%"
+		(property "Value" "270 Ω"
 			(at 241.3 182.88 0)
 			(effects
@@
 			)
 		)
-		(property "Value" "1 kΩ ±1%"
+		(property "Value" "1 kΩ"
 			(at 234.95 150.495 90)
 			(effects
@@
 			)
 		)
-		(property "Value" "220 Ω ±5%"
+		(property "Value" "220 Ω"
 			(at 342.9 199.39 90)
 			(effects
@@
 			)
 		)
-		(property "Value" "270 Ω ±5%"
+		(property "Value" "270 Ω"
 			(at 326.39 166.37 90)
 			(effects
@@
 			)
 		)
-		(property "Value" "10 kΩ ±5%"
+		(property "Value" "10 kΩ"
 			(at 97.79 180.34 90)
 			(effects
@@
 		(fields_autoplaced yes)
 		(property "Reference" "D1"
-			(at 321.31 205.74 0)
+			(at 330.2 204.4699 90)
 			(effects
 				(font
 					(size 1.27 1.27)
 				)
+				(justify right)
 			)
 		)
-		(property "Value" "D"
-			(at 323.85 205.74 0)
+		(property "Value" "1N5819"
+			(at 330.2 207.0099 90)
 			(effects
 				(font
 					(size 1.27 1.27)
 				)
+				(justify right)
 			)
 		)
@@
 			)
 		)
-		(property "Value" "270 Ω ±5%"
+		(property "Value" "270 Ω"
 			(at 311.15 175.2599 0)
 			(effects
@@
 			)
 		)
-		(property "Value" "47 kΩ ±5%"
+		(property "Value" "47 kΩ"
 			(at 95.25 162.56 90)
 			(effects
@@
 			)
 		)
-		(property "Value" "1 kΩ ±1%"
+		(property "Value" "1 kΩ"
 			(at 229.87 172.085 90)
 			(effects
@@
 			)
 		)
-		(property "Value" "4.7 kΩ ±1%"
+		(property "Value" "4.7 kΩ"
 			(at 248.92 69.85 90)
 			(effects
@@
 			)
 		)
-		(property "Value" "100 kΩ ±5%"
+		(property "Value" "100 kΩ"
 			(at 241.3 69.85 90)
 			(effects
@@
 			)
 		)
-		(property "Value" "4.7 kΩ ±1%"
+		(property "Value" "4.7 kΩ"
 			(at 252.73 138.4299 0)
 			(effects
@@
 			)
 		)
-		(property "Value" "3.3 kΩ ±5%"
+		(property "Value" "3.3 kΩ"
 			(at 58.42 123.19 0)
 			(effects
@@
 			)
 		)
-		(property "Value" "1 kΩ ±1%"
+		(property "Value" "1 kΩ"
 			(at 316.23 241.2999 0)
 			(effects
@@
 			)
 		)
-		(property "Value" "100 Ω ±1%"
+		(property "Value" "100 Ω"
 			(at 386.08 179.07 0)
 			(effects
@@
 		(fields_autoplaced yes)
 		(property "Reference" "D3"
-			(at 243.84 173.99 90)
+			(at 243.84 173.9899 90)
 			(effects
 				(font
@@
 			)
 		)
-		(property "Value" "D"
-			(at 243.84 176.53 90)
+		(property "Value" "1N5819"
+			(at 243.84 176.5299 90)
 			(effects
 				(font
@@
 			)
 		)
-		(property "Value" "22 Ω ±5%"
+		(property "Value" "22 Ω"
 			(at 76.2 162.56 90)
 			(effects
@@
 			)
 		)
-		(property "Value" "1 kΩ ±1%"
+		(property "Value" "1 kΩ"
 			(at 147.32 157.48 90)
 			(effects
@@
 			)
 		)
-		(property "Value" "1 kΩ ±1%"
+		(property "Value" "1 kΩ"
 			(at 229.87 161.925 90)
 			(effects
@@
 			)
 		)
-		(property "Value" "1 Ω ±5%"
+		(property "Value" "1 Ω"
 			(at 368.3 177.8 90)
 			(effects
@@
 			)
 		)
-		(property "Value" "47 Ω ±1%"
+		(property "Value" "47 Ω"
 			(at 218.44 158.115 90)
 			(effects
